Commit message: Get images to python node

File: models/stereo_cam/dimensions.xacro (robot description, xacro)
@@ -15,5 +15,5 @@
     <!-- Cameras -->
     <!-- <xacro:property name="ipd" value="${64.0 * 0.01}"/> -->
-    <xacro:property name="ipd" value="0.3"/>
+    <xacro:property name="ipd" value="0.5"/>
     <xacro:property name="cam_size" value="0.05"/>
 </robot>

Commit message: Disparity maps

File: models/stereo_cam/dimensions.xacro (robot description, xacro)
@@ -2,7 +2,7 @@
 <robot xmlns:xacro="http://www.ros.org/wiki/xacro">
     <!-- Body -->
-    <xacro:property name="body_x" value="0.15"/>
+    <xacro:property name="body_x" value="0.07"/>
     <xacro:property name="body_y" value="${body_x}"/>
-    <xacro:property name="body_z" value="1.5"/>
+    <xacro:property name="body_z" value="1.1"/>
     <xacro:property name="body_dim" value="${body_x} ${body_y} ${body_z}"/>
     <!-- Arm -->
@@ -15,5 +15,5 @@
     <!-- Cameras -->
     <!-- <xacro:property name="ipd" value="${64.0 * 0.01}"/> -->
-    <xacro:property name="ipd" value="0.5"/>
+    <xacro:property name="ipd" value="0.15"/>
     <xacro:property name="cam_size" value="0.05"/>
 </robot>

File: models/stereo_cam/gazebo.xacro (robot description, xacro)
@@ -20,12 +20,12 @@
     <!-- Camera R -->
     <gazebo reference="camera_r_link">
-        <sensor type="camera" name="camera_r">
-            <update_rate>20</update_rate>
+        <sensor type="camera" name="stereo/right">
+            <update_rate>30</update_rate>
             <visualize>true</visualize>
             <camera name="cam_r">
-                <horizontal_fov>1.3962634</horizontal_fov>
+                <horizontal_fov>1.04699999</horizontal_fov>
                 <image>
-                    <width>800</width>
-                    <height>800</height>
+                    <width>720</width>
+                    <height>480</height>
                     <format>R8G8B8</format>
                 </image>
@@ -49,12 +49,12 @@
     <!-- Camera L -->
     <gazebo reference="camera_l_link">
-        <sensor type="camera" name="camera_l">
+        <sensor type="camera" name="stereo/left">
             <update_rate>30</update_rate>
             <visualize>true</visualize>
             <camera name="cam_l">
-                <horizontal_fov>1.3962634</horizontal_fov>
+                <horizontal_fov>1.04699999</horizontal_fov>
                 <image>
-                    <width>800</width>
-                    <height>800</height>
+                    <width>720</width>
+                    <height>480</height>
                     <format>R8G8B8</format>
                 </image>

Commit message: Disparity map

File: models/stereo_cam/dimensions.xacro (robot description, xacro)
@@ -4,5 +4,5 @@
     <xacro:property name="body_x" value="0.07"/>
     <xacro:property name="body_y" value="${body_x}"/>
-    <xacro:property name="body_z" value="1.1"/>
+    <xacro:property name="body_z" value="1"/>
     <xacro:property name="body_dim" value="${body_x} ${body_y} ${body_z}"/>
     <!-- Arm -->
@@ -14,6 +14,5 @@
     <xacro:property name="arm_vis2_dim" value="${arm_thickness} ${arm_span} ${arm_thickness}"/>
     <!-- Cameras -->
-    <!-- <xacro:property name="ipd" value="${64.0 * 0.01}"/> -->
-    <xacro:property name="ipd" value="0.15"/>
+    <xacro:property name="ipd" value="0.065"/>
     <xacro:property name="cam_size" value="0.05"/>
 </robot>

File: models/stereo_cam/stereo_cam.urdf.xacro (robot description, xacro)
@@ -68,5 +68,5 @@
     </link>
     <joint name="camera_r_fix" type="fixed">
-        <origin xyz = "0 ${ipd/2} 0"/>
+        <origin xyz = "${arm_thickness/2} -${ipd/2} 0"/>
         <parent link = "arm"/>
         <child link = "camera_r_link"/>
@@ -82,7 +82,14 @@
     </link>
     <joint name="camera_l_fix" type="fixed">
-        <origin xyz = "0 -${ipd/2} 0"/>
+        <origin xyz = "${arm_thickness/2} ${ipd/2} 0"/>
         <parent link = "arm"/>
         <child link = "camera_l_link"/>
     </joint>
+    <!-- Camera Midpoint (PCL Reference) -->
+    <link name="camera_midpoint"></link>
+    <joint name="camera_midpoint_fix" type="fixed">
+        <origin xyz = "${arm_thickness/2} 0 0"/>
+        <parent link = "arm"/>
+        <child link = "camera_midpoint"/>
+    </joint>
 </robot>
