Commit message: Figured out DAE files and Blender

File: models/simple_targets/cubesat.urdf.xacro (robot description, xacro)
@@ -1,4 +1,4 @@
 <?xml version='1.0'?>
-<robot xmlns:xacro="http://www.ros.org/wiki/xacro" name="stereo">
+<robot xmlns:xacro="http://www.ros.org/wiki/xacro" name="cubesat">
     <xacro:include filename="dimensions.xacro"/>
     <xacro:include filename="macros.xacro"/>

File: models/simple_targets/gazebo.xacro (robot description, xacro)
@@ -9,3 +9,7 @@
         </plugin>
     </gazebo>
+    <!-- Body Material -->
+    <!-- <gazebo reference="body">
+        <material>MarkersTexture</material>
+    </gazebo> -->
 </robot>
