Commit message: Aruco Cube simulation

File: models/simple_targets/gazebo.xacro (robot description, xacro)
@@ -9,7 +9,7 @@
         </plugin>
     </gazebo>
-    <!-- Body Material -->
-    <!-- <gazebo reference="body">
-        <material>MarkersTexture</material>
-    </gazebo> -->
+    <!-- Gravity -->
+    <gazebo reference="body">
+        <gravity>0</gravity>
+    </gazebo>
 </robot>

File: models/simple_targets/marker_cube.urdf.xacro (robot description, xacro)
@@ -3,6 +3,5 @@
     <xacro:include filename="dimensions.xacro"/>
     <xacro:include filename="macros.xacro"/>
-    <!-- World -->
-    <link name="world"></link>
+    <xacro:include filename="gazebo.xacro"/>
     <!-- Body -->
     <link name="body">
@@ -14,5 +13,5 @@
         <visual name="body_visual_cube">
             <geometry>
-                <mesh filename="/home/frank20a/dev-ws/models/media/meshes/marker_cube_test.dae" scale="10 10 10"/>
+                <mesh filename="/home/frank20a/dev-ws/models/media/meshes/marker_box.dae"/>
             </geometry>
         </visual>
@@ -21,9 +20,3 @@
         </xacro:inertial_box>
     </link>
-    <joint name="body_fix" type="fixed">
-        <origin xyz="0 0 ${cube_z * U + 0.05}"/>
-        <parent link="world"/>
-        <child link="body"/>
-    </joint>
-    <xacro:include filename="gazebo.xacro"/>
 </robot>
