Commit message: Fixed some models

File: models/simple_targets/marker_cube.urdf.xacro (robot description, xacro)
@@ -13,5 +13,5 @@
         <visual name="body_visual_cube">
             <geometry>
-                <mesh filename="/home/frank20a/dev-ws/models/media/meshes/marker_box.dae"/>
+                <mesh filename="/home/frank20a/dev-ws/models/simple_targets/ship1/marker_box.dae"/>
             </geometry>
         </visual>

Commit message: Minor Fixes + New temp material to fix marker orientation ~ Changed stuff a bit to support target visualization on rviz

File: models/simple_targets/marker_cube.urdf.xacro (robot description, xacro)
@@ -4,6 +4,7 @@
     <xacro:include filename="macros.xacro"/>
     <xacro:include filename="gazebo.xacro"/>
+    <link name="marker_3"></link>
     <!-- Body -->
-    <link name="body">
+    <link name="target_body">
         <collision name="body_collision">
             <geometry>
@@ -20,3 +21,8 @@
         </xacro:inertial_box>
     </link>
+    <joint name="body_fix" type="fixed">
+        <origin xyz="0 0 0" rpy="${-pi/2} ${pi} ${-pi/2}"/>
+        <parent link="marker_3"/>
+        <child link="target_body"/>
+    </joint>
 </robot>

Commit message: Slider Model

File: models/simple_targets/marker_cube.urdf.xacro (robot description, xacro)
@@ -22,5 +22,4 @@
     </link>
     <joint name="body_fix" type="fixed">
-        <!-- <origin xyz="0 0 0" rpy="${-pi/2} ${pi} ${-pi/2}"/> -->
         <parent link="estimated_pose"/>
         <child link="target_body"/>
