Commit message: Added flashlight to chaser

File: models/chaser/gazebo.xacro (robot description, xacro)
@@ -19,4 +19,22 @@
     <!-- Camera -->
     <gazebo reference="camera">
+        <light name='flashlight' type='spot'>
+            <pose>0 0 0 -3.14159 -1.57059 3.14159</pose>
+            <diffuse>0.5 0.5 0.5 1</diffuse>
+            <specular>0.1 0.1 0.1 1</specular>
+            <direction>0 0 -1</direction>
+            <attenuation>
+                <range>30</range>
+                <constant>0.35</constant>
+                <linear>0.01</linear>
+                <quadratic>0.001</quadratic>
+            </attenuation>
+            <cast_shadows>0</cast_shadows>
+            <spot>
+                <inner_angle>0.6</inner_angle>
+                <outer_angle>1</outer_angle>
+                <falloff>1</falloff>
+            </spot>
+        </light>
         <sensor type="camera" name="sim_camera">
             <update_rate>60</update_rate>

File: models/simple_targets/marker_cube.urdf.xacro (robot description, xacro)
@@ -4,5 +4,5 @@
     <xacro:include filename="macros.xacro"/>
     <xacro:include filename="gazebo.xacro"/>
-    <link name="marker_3"></link>
+    <link name="estimated_pose"></link>
     <!-- Body -->
     <link name="target_body">
@@ -23,5 +23,5 @@
     <joint name="body_fix" type="fixed">
         <origin xyz="0 0 0" rpy="${-pi/2} ${pi} ${-pi/2}"/>
-        <parent link="marker_3"/>
+        <parent link="estimated_pose"/>
         <child link="target_body"/>
     </joint>

Commit message: Fixes on simulation world

File: models/chaser/gazebo.xacro (robot description, xacro)
@@ -54,5 +54,5 @@
                     <type>gaussian</type>
                     <mean>0.0</mean>
-                    <stddev>0.007</stddev>
+                    <stddev>0.01</stddev>
                 </noise>
             </camera>

File: models/simple_targets/marker_cube.urdf.xacro (robot description, xacro)
@@ -22,5 +22,5 @@
     </link>
     <joint name="body_fix" type="fixed">
-        <origin xyz="0 0 0" rpy="${-pi/2} ${pi} ${-pi/2}"/>
+        <!-- <origin xyz="0 0 0" rpy="${-pi/2} ${pi} ${-pi/2}"/> -->
         <parent link="estimated_pose"/>
         <child link="target_body"/>
