Commit message: Fixed Camera Frame Miss-alignment

File: models/chaser/chaser.urdf.xacro (robot description, xacro)
@@ -76,3 +76,12 @@
         <child link = "camera"/>
     </joint>
+    <link name="camera_optical"></link>
+    <joint name="camera_optical_joint" type="fixed">
+        <!-- these values have to be these values otherwise the gazebo camera
+            image won't be aligned properly with the frame it is supposedly
+            originating from -->
+        <origin xyz="0 0 0" rpy="${-pi/2} 0 ${-pi/2}"/>
+        <parent link="camera"/>
+        <child link="camera_optical"/>
+      </joint>
 </robot>

File: models/chaser/gazebo.xacro (robot description, xacro)
@@ -40,5 +40,5 @@
             </camera>
             <plugin name="camera_plugin" filename="libgazebo_ros_camera.so">
-                <frameName>camera</frameName>
+                <frameName>camera_optical</frameName>
                 <min_depth>0.1</min_depth>
                 <max_depth>500</max_depth>

Commit message: Multiple Chasers

File: models/chaser/chaser.urdf.xacro (robot description, xacro)
@@ -3,7 +3,6 @@
     <xacro:include filename="dimensions.xacro"/>
     <xacro:include filename="macros.xacro"/>
-    <xacro:include filename="gazebo.xacro"/>
     <!-- World -->
-    <link name="world"></link>
+    <!-- <link name="world"></link> -->
     <!-- Body -->
     <link name="body">
@@ -57,9 +56,9 @@
         </xacro:inertial_box>
     </link>
-    <joint name="body_fix" type="fixed">
-        <origin xyz="0 0 0.75"/>
+    <!-- <joint name="body_fix" type="fixed">
+        <origin xyz="0 0 0"/>
         <parent link="world"/>
         <child link="body"/>
-    </joint>
+    </joint> -->
     <!-- Camera L -->
     <link name="camera">
@@ -84,4 +83,5 @@
         <parent link="camera"/>
         <child link="camera_optical"/>
-      </joint>
+    </joint>
+    <xacro:include filename="gazebo.xacro"/>
 </robot>

File: models/chaser/gazebo.xacro (robot description, xacro)
@@ -2,4 +2,7 @@
 <robot xmlns:xacro="http://www.ros.org/wiki/xacro">
     <xacro:include filename="macros.xacro"/>
+    <gazebo>
+        <static>true</static>
+    </gazebo>
     <!-- Materials -->
     <gazebo reference="body">
@@ -11,8 +14,14 @@
     <!-- Plugins -->
     <gazebo>
-        <plugin name="gazebo_ros_joint_state_publisher"
+        <!-- <plugin name="gazebo_ros_joint_state_publisher"
             filename="libgazebo_ros_joint_state_publisher.so">
             <update_rate>30</update_rate>
-            <joint_name>body_fix</joint_name>
+            <joint_name>camera_fix</joint_name>
+        </plugin> -->
+        <plugin name="p3d" filename="libgazebo_ros_p3d.so">
+            <frame_name>world</frame_name>
+            <body_name>body</body_name>
+            <topic_name>odom</topic_name>
+            <update_rate>30.0</update_rate>
         </plugin>
     </gazebo>
@@ -37,5 +46,5 @@
             </spot>
         </light>
-        <sensor type="camera" name="sim_camera">
+        <sensor type="camera" name="front_cam">
             <update_rate>60</update_rate>
             <visualize>true</visualize>

Commit message: Target Lock

File: models/chaser/chaser.urdf.xacro (robot description, xacro)
@@ -3,6 +3,6 @@
     <xacro:include filename="dimensions.xacro"/>
     <xacro:include filename="macros.xacro"/>
-    <!-- World -->
-    <!-- <link name="world"></link> -->
+    <!-- Dummy root link -->
+    <!-- <link name="root"></link> -->
     <!-- Body -->
     <link name="body">
@@ -56,7 +56,7 @@
         </xacro:inertial_box>
     </link>
-    <!-- <joint name="body_fix" type="fixed">
+    <!-- <joint name="root_fix" type="fixed">
         <origin xyz="0 0 0"/>
-        <parent link="world"/>
+        <parent link="root"/>
         <child link="body"/>
     </joint> -->

File: models/simple_targets/gazebo.xacro (robot description, xacro)
@@ -8,4 +8,14 @@
             <joint_name>body_fix</joint_name>
         </plugin>
+      <plugin name="controller_plugin" filename="libgazebo_ros_force.so">
+          <link_name>body</link_name>
+          <force_frame>link</force_frame>
+      </plugin>
+      <plugin name="p3d" filename="libgazebo_ros_p3d.so">
+          <frame_name>world</frame_name>
+          <body_name>body</body_name>
+          <topic_name>odom</topic_name>
+          <update_rate>30.0</update_rate>
+      </plugin>
     </gazebo>
     <!-- Gravity -->

Commit message: Added grabber to chaser

File: models/chaser/chaser.urdf.xacro (robot description, xacro)
@@ -27,4 +27,5 @@
                 <cylinder radius="${leg_r}" length="${leg_len}"/>
             </geometry>
+            <material name="white"/>
         </visual>
         <visual name="leg_2">
@@ -33,4 +34,5 @@
                 <cylinder radius="${leg_r}" length="${leg_len}"/>
             </geometry>
+            <material name="white"/>
         </visual>
         <visual name="leg_3">
@@ -39,4 +41,5 @@
                 <cylinder radius="${leg_r}" length="${leg_len}"/>
             </geometry>
+            <material name="white"/>
         </visual>
         <visual name="leg_4">
@@ -45,4 +48,5 @@
                 <cylinder radius="${leg_r}" length="${leg_len}"/>
             </geometry>
+            <material name="white"/>
         </visual>
         <visual name="head_vis">
@@ -51,4 +55,5 @@
                 <cylinder radius="${head_r}" length="${head_len}"/>
             </geometry>
+            <material name="white"/>
         </visual>
         <xacro:inertial_box mass="30.0" x="${body_x}" y="${body_y}" z="${body_z}">
@@ -61,5 +66,5 @@
         <child link="body"/>
     </joint> -->
-    <!-- Camera L -->
+    <!-- Camera -->
     <link name="camera">
         <visual>
@@ -68,4 +73,5 @@
                 <box size="${cam_size} ${cam_size} ${cam_size}"/>
             </geometry>
+            <material name="red"/>
         </visual>
     </link>
@@ -84,4 +90,24 @@
         <child link="camera_optical"/>
     </joint>
+    <!-- Grabber -->
+    <link name="grabber">
+        <visual>
+            <geometry>
+                <cylinder radius="0.01" length="${0.35 - body_x/2}"/>
+            </geometry>
+            <material name="black"/>
+        </visual>
+        <visual>
+            <origin xyz="0 0 ${-(0.35 - body_x/2)/2}"/>
+            <geometry>
+                <sphere radius="0.02"/>
+            </geometry>
+        </visual>
+    </link>
+    <joint name="grabber_fix" type="fixed">
+        <origin xyz="${body_x/2} 0 0" rpy="0 ${-pi/2} 0"/>
+        <parent link="body"/>
+        <child link="grabber"/>
+    </joint>
     <xacro:include filename="gazebo.xacro"/>
 </robot>

File: models/chaser/gazebo.xacro (robot description, xacro)
@@ -8,4 +8,7 @@
     <gazebo reference="camera">
         <material>Gazebo/Red</material>
+    </gazebo>
+    <gazebo reference="grabber">
+        <material>Gazebo/Blue</material>
     </gazebo>
     <!-- Plugins -->
