Commit message: Slider Controller

File: models/slider/slider.urdf.xacro (robot description, xacro)
@@ -12,5 +12,5 @@
             <origin rpy="0 0 ${pi}"/>
             <geometry>
-                <mesh filename="/home/frank20a/dev-ws/models/slider/slider_model_05.stl"/>
+                <mesh filename="/home/frank20a/dev-ws/models/slider/slider_model_05.dae"/>
             </geometry>
         </visual>
