Commit message: Moved models

File: data/models/chaser/gazebo.xacro (robot description, xacro)
@@ -51,5 +51,5 @@
         </light>
         <sensor type="camera" name="front_cam">
-            <update_rate>60</update_rate>
+            <update_rate>25</update_rate>
             <visualize>true</visualize>
             <camera name="cam">

File: data/models/simple_targets/cubesat.urdf.xacro (robot description, xacro)
@@ -4,7 +4,7 @@
     <xacro:include filename="macros.xacro"/>
     <!-- World -->
-    <link name="world"></link>
+    <link name="estimated_pose"></link>
     <!-- Body -->
-    <link name="body">
+    <link name="target_body">
         <collision name="body_collision">
             <geometry>
@@ -35,4 +35,10 @@
             </geometry>
         </visual>
+        <visual name="body_visual_cube">
+            <origin rpy="0 0 ${pi/2}"/>
+            <geometry>
+                <mesh filename="/home/frank20a/dev-ws/data/models/simple_targets/ship2/cubesat.dae"/>
+            </geometry>
+        </visual>
         <xacro:inertial_box mass="1.25" x="${cube_x*U}" y="${cube_y*U}" z="${cube_z*U}">
             <origin xyz="0 0 0"/>
@@ -40,7 +46,10 @@
     </link>
     <joint name="body_fix" type="fixed">
-        <origin xyz="0 0 ${cube_z * U + 0.05}"/>
-        <parent link="world"/>
-        <child link="body"/>
+        <!-- <origin xyz="0 0 ${cube_z * U + 0.05}"/>
+        <parent link="world"/> -->
+        <origin rpy="0 0 ${pi/2}"/>
+        <parent link="estimated_pose"/>
+        <child link="target_body"/>
     </joint>
+    <xacro:include filename="gazebo.xacro"/>
 </robot>

File: data/models/simple_targets/marker_cube.urdf.xacro (robot description, xacro)
@@ -14,5 +14,5 @@
         <visual name="body_visual_cube">
             <geometry>
-                <mesh filename="/home/frank20a/dev-ws/models/simple_targets/ship1/marker_box.dae"/>
+                <mesh filename="/home/frank20a/dev-ws/data/models/simple_targets/ship1/marker_box.dae"/>
             </geometry>
         </visual>

File: data/models/slider/slider.urdf.xacro (robot description, xacro)
@@ -12,5 +12,5 @@
             <origin rpy="0 0 ${pi}"/>
             <geometry>
-                <mesh filename="/home/frank20a/dev-ws/models/slider/slider_model_05.dae"/>
+                <mesh filename="/home/frank20a/dev-ws/data/models/slider/slider_model_05.dae"/>
             </geometry>
         </visual>

Commit message: Work

File: data/models/chaser/gazebo.xacro (robot description, xacro)
@@ -32,5 +32,5 @@
     <!-- Camera -->
     <gazebo reference="camera">
-        <!-- <light name='flashlight' type='spot'>
+        <light name='flashlight' type='spot'>
             <pose>0 0 0 -3.14159 -1.57059 3.14159</pose>
             <diffuse>0.5 0.5 0.5 1</diffuse>
@@ -49,5 +49,5 @@
                 <falloff>1</falloff>
             </spot>
-        </light> -->
+        </light>
         <sensor type="camera" name="front_cam">
             <update_rate>30</update_rate>

File: data/models/simple_targets/cubesat.urdf.xacro (robot description, xacro)
@@ -29,8 +29,8 @@
             </geometry>
         </visual>
-        <visual name="body_visual_panel_left">
-            <origin xyz="0 ${-(cube_y*U + panel_y)/2 - arm} 0" rpy="0 1.0472 0"/>
+        <visual name="sphere">
+            <origin xyz="0 0 ${cube_z/15}" rpy="0 0 0"/>
             <geometry>
-                <box size="${panel_dim}"/>
+                <sphere radius="${cube_z / 20}"/>
             </geometry>
         </visual>
@@ -48,5 +48,5 @@
         <!-- <origin xyz="0 0 ${cube_z * U + 0.05}"/>
         <parent link="world"/> -->
-        <origin rpy="0 0 ${pi/2}"/>
+        <origin rpy="${pi/2} ${pi/2} 0"/>
         <parent link="estimated_pose"/>
         <child link="target_body"/>
